File: PCBs/right_finished.kicad_pcb (KiCad board)
At the start: 2 copper layers, 147.2 x 118.7 mm, 68 parts

Commit message: file(3D): move to the root folder / feat(add): Add image to the PCBs
Parts:
- added G***: LOGO, PCBs:flag, F.Cu at (226.5, 141.8)
